File: PCB/dd-pcb.kicad_sch (KiCad schematic)
At the start: 12 parts, among them J1 Conn_01x04_Pin, J2 Conn_01x02_Pin, J3 Conn_01x04_Pin, J4 Conn_01x02_Pin, U1 SeeedStudio ESP32C3

Commit message: Changed components
Parts:
- removed J3: Conn_01x04_Pin, Connector_PinSocket_2.54mm:PinSocket_1x04_P2.54mm_Vertical, symbol Connector:Conn_01x04_Pin
- added LED_Strip: Conn_02x08_Odd_Even, symbol Connector_Generic:Conn_02x07_Odd_Even
- added Mode: Conn_01x03_Pin, symbol Connector:Conn_01x03_Pin
- added R10: 10K, Resistor_SMD:R_0805_2012Metric, symbol Device:R
- added R2, R3, R4, R5, R6, R7, R8: 220R, Resistor_SMD:R_0805_2012Metric, symbol Device:R
- added R9: 100K, Resistor_SMD:R_0805_2012Metric, symbol Device:R
- renumbered J1 to AudioModule, J4 to BATT
Connections:
- net +3V3: now also R9.2
- net GND: now also U1.20 (GND), LED_Strip.10 (Pin_10), LED_Strip.12 (Pin_12), LED_Strip.14 (Pin_14), LED_Strip.2 (Pin_2), LED_Strip.4 (Pin_4), LED_Strip.6 (Pin_6), LED_Strip.8 (Pin_8), R10.1
- net at R1.2: now also U1.1 (GPIO2_A0_D0); no longer U1.2 (GPIO3_A1_D1)
- net LED6: now reaches U1.10 (GPIO9_D9_MISO)
- net LED6: now also R8.1
- net LED5: now reaches U1.11 (GPIO10_D10_MOSI)
- net LED5: now also R7.1
- net LED1: now reaches U1.3 (GPIO4_A2_D2)
- net LED1: now also R3.1
- net LED2: now reaches U1.4 (GPIO5_A2_D2)
- net LED2: now also R4.1
- net LED3: now reaches U1.5 (GPIO6_SDA_D4)
- net LED3: now also R5.1
- net LED4: now reaches U1.6 (GPIO7_SCL_D5)
- net LED4: now also R6.1
- net IN0: now reaches U1.9 (GPIO8_D8_SCK)
- net IN0: now also Mode.2 (Pin_2)
- new net: LED_Strip.3 (Pin_3), R3.2
- new net: Mode.1 (Pin_1), R9.1
- new net: Mode.3 (Pin_3), R10.2
- new net: LED_Strip.1 (Pin_1), R2.2
- new net: LED_Strip.11 (Pin_11), R7.2
- new net: LED_Strip.13 (Pin_13), R8.2
- new net: LED_Strip.5 (Pin_5), R4.2
- new net: LED_Strip.7 (Pin_7), R5.2
- new net: LED_Strip.9 (Pin_9), R6.2
- new net LED0: R2.1, U1.2 (GPIO3_A1_D1)
- no-connect marks 4 -> 3
Other:
- moved on the sheet: AudioModule, C1, C3, J2, R1
